Commit message: fixed some vrp related bugs, added ground contraint and working on terrain

File: python/py_dcm_vrp_planner/terrains/stairs.urdf (robot description, URDF)
Before this commit: robot stairs, 7 links, 6 joints
Links:
- link first_step_link: geometry collision box size=0.2 1.0 .1; visual box size=0.2 1.0 .1
- link fourth_step_link: geometry collision box size=0.6 1.0 .4; visual box size=0.6 1.0 .4
- link second_step_link: geometry collision box size=0.2 1.0 .2; visual box size=0.2 1.0 .2
- link sixth_step_link: geometry collision box size=0.6 1.0 .4; visual box size=.6 1.0 .4
- link third_step_link: geometry collision box size=0.4 1.0 .3; visual box size=0.4 1.0 .3
Joints:
- joint first_to_second_step: origin (none) -> xyz=0 0 0 
- joint fourth_to_fifth_step_left: parent fourth_step_link -> first_step_link
- joint fourth_to_fifth_step_right: parent fourth_step_link -> first_step_link
- joint second_to_third_step: parent second_step_link -> first_step_link
- joint third_to_fourth_step: parent third_step_link -> first_step_link

Commit message: implemented split dcm with gurobi and cvxpy. gurobi not working. to be debuged

File: python/py_dcm_vrp_planner/terrains/stairs.urdf (robot description, URDF)
Before this commit: robot stairs, 7 links, 6 joints
Links:
- added link ground_link, mass .0; collision box size=1.8 1.0 .05; visual box size=1.8 1.0 .05
Joints:
- added joint ground_to_first_step: type fixed, parent ground_link, child first_step_link

Commit message: updated trajectory generator

File: python/py_dcm_vrp_planner/terrains/stairs.urdf (robot description, URDF)
Before this commit: robot stairs, 8 links, 7 joints
Links:
- removed link fifth_step_link_left
- removed link fifth_step_link_right
- removed link fourth_step_link
- removed link sixth_step_link
- removed link third_step_link
- link first_step_link: geometry collision box size=0.7 2.0 .1; visual box size=0.7 2.0 .1
- link ground_link: geometry collision box size=1.6 1.0 .1; visual box size=1.6 1.0 .1
- link second_step_link: geometry collision box size=0.2 2.0 .1; visual box size=0.2 2.0 .1
Joints:
- removed joint fifth_step_left_to_sixth
- removed joint fourth_to_fifth_step_left
- removed joint fourth_to_fifth_step_right
- removed joint second_to_third_step
- removed joint third_to_fourth_step
